File: panel_rp2354_20x20_ir-red_v0p4/panel_led.kicad_sch (KiCad schematic)
At the start: 420 parts

Commit message: IR-red panel v0.4r2: checkerboard, 33/56 Ω 0.2 W 0402 column resistors
- LED banks: T2 -> IR (C6879329), T3 -> red (C2852592); red is now T0+T3
  (checkerboard, firmware channels 0 and 3), IR T1+T2. BOM-only change.
- R9-R28: Resistor_SMD:R_0201_0603Metric -> R_0402_1005Metric, same
  rotation and side. Red banks 33 Ω (Panasonic ERJ-PA2F33R0X, C427231),
  IR banks 56 Ω (ERJ-PA2F56R0X, C427233; 0 stock at JLC on 2026-09-26,
  alternates listed in CHANGES-v0p4r2.md). Vishay CRCW-HP codes noted.
- Layout: nine resistor centres nudged 0.03-0.20 mm, ten vias moved, six
  short track re-routes so every 0402 pad has >= 0.135 mm to foreign
  copper; no driver or other part moved. DRC at 0.127 mm clearance has
  the same 68 pre-existing 0.125 mm netclass items as v0.4r1, 0
  unconnected, plus 19 courtyard overlaps (0402 vs SOT-23-5 courtyards).
- production/v0p4r2 regenerated with Fabrication Toolkit 5.3.1; board rev
  v0.4.2. Scripts used are in tools/column_resistors_0402 and apply to
  the four-color and v0.3 boards (identical layouts).

Co-Authored-By: Claude Fable 5.1 <noreply@anthropic.com>
Parts:
- D121, D122, D123, D124, D125, D126, D127, D128, D129, D130, D131, D132, D133, D134, D135, D136, D137, D138, D139, D140, D201, D202, D203, D204, D205, D206, D207, D208, D209, D210, D211, D212, D213, D214, D215, D216, D217, D218, D219, D220, D281, D282, D283, D284, D285, D286, D287, D288, D289, D290, D291, D292, D293, D294, D295, D296, D297, D298, D299, D300, D361, D362, D363, D364, D365, D366, D367, D368, D369, D370, D371, D372, D373, D374, D375, D376, D377, D378, D379, D380, D41, D42, D43, D44, D45, D46, D47, D48, D49, D50, D51, D52, D53, D54, D55, D56, D57, D58, D59, D60: LCSC Part # C2852592 -> C6879329
- D141, D142, D143, D144, D145, D146, D147, D148, D149, D150, D151, D152, D153, D154, D155, D156, D157, D158, D159, D160, D221, D222, D223, D224, D225, D226, D227, D228, D229, D230, D231, D232, D233, D234, D235, D236, D237, D238, D239, D240, D301, D302, D303, D304, D305, D306, D307, D308, D309, D310, D311, D312, D313, D314, D315, D316, D317, D318, D319, D320, D381, D382, D383, D384, D385, D386, D387, D388, D389, D390, D391, D392, D393, D394, D395, D396, D397, D398, D399, D400, D61, D62, D63, D64, D65, D66, D67, D68, D69, D70, D71, D72, D73, D74, D75, D76, D77, D78, D79, D80: LCSC Part # C6879329 -> C2852592
- R10, R11, R14, R15, R18, R19, R22, R23, R26, R27: footprint Resistor_SMD:R_0201_0603Metric -> Resistor_SMD:R_0402_1005Metric; LCSC Part # C77623 -> C427233
- R12, R13, R16, R17, R20, R21, R24, R25, R28, R9: footprint Resistor_SMD:R_0201_0603Metric -> Resistor_SMD:R_0402_1005Metric; LCSC Part # C77623 -> C427231

Commit message: v0.4r2: column resistors 22 Ω red / 47 Ω IR (in-stock 0.2 W 0402 parts)
Red banks R_T0/R_T3: Vishay CRCW040222R0FKEDHP (C313374); IR banks
R_T1/R_T2: ROHM ESR01MZPF47R0 (C5736551). Chosen to maximise LED current
within the 0.2 W rating using parts in stock (56 Ω had none). Model:
red ≈87 mA at 75 % of rating, IR ≈64 mA at 88 %; all-on row current
1.29 A, 5 V droop ≈0.65 V over the 45 µs pulse. Full-field 5 V supply
current is ≈0.9 × row current ≈ 1.16 A per panel; the analysis doc's
"≈50 mA" figure is wrong by ×20 — power path to be checked.

Production BOM regenerated; positions unchanged. Notes and scripts updated.

Co-Authored-By: Claude Fable 5.1 <noreply@anthropic.com>
Parts:
- R10, R11, R14, R15, R18, R19, R22, R23, R26, R27: LCSC Part # C427233 -> C5736551
- R12, R13, R16, R17, R20, R21, R24, R25, R28, R9: LCSC Part # C427231 -> C313374
Changed lines of the file:
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@@
 			)
 		)
-		(property "LCSC Part #" "C427231"
+		(property "LCSC Part #" "C313374"
 			(at 83.82 53.34 0)
 			(hide yes)
@@
 			)
 		)
-		(property "LCSC Part #" "C427233"
+		(property "LCSC Part #" "C5736551"
 			(at 66.04 53.34 0)
 			(hide yes)
@@
 			)
 		)
-		(property "LCSC Part #" "C427231"
+		(property "LCSC Part #" "C313374"
 			(at 154.94 53.34 0)
 			(hide yes)
@@
 			)
 		)
-		(property "LCSC Part #" "C427231"
+		(property "LCSC Part #" "C313374"
 			(at 369.57 53.34 0)
 			(hide yes)
@@
 			)
 		)
-		(property "LCSC Part #" "C427233"
+		(property "LCSC Part #" "C5736551"
 			(at 279.4 53.34 0)
 			(hide yes)
@@
 			)
 		)
-		(property "LCSC Part #" "C427233"
+		(property "LCSC Part #" "C5736551"
 			(at 261.62 53.34 0)
 			(hide yes)
@@
 			)
 		)
-		(property "LCSC Part #" "C427233"
+		(property "LCSC Part #" "C5736551"
 			(at 208.28 53.34 0)
 			(hide yes)
@@
 			)
 		)
-		(property "LCSC Part #" "C427231"
+		(property "LCSC Part #" "C313374"
 			(at 226.06 53.34 0)
 			(hide yes)
@@
 			)
 		)
-		(property "LCSC Part #" "C427233"
+		(property "LCSC Part #" "C5736551"
 			(at 119.38 53.34 0)
 			(hide yes)
@@
 			)
 		)
-		(property "LCSC Part #" "C427233"
+		(property "LCSC Part #" "C5736551"
 			(at 351.79 53.34 0)
 			(hide yes)
@@
 			)
 		)
-		(property "LCSC Part #" "C427231"
+		(property "LCSC Part #" "C313374"
 			(at 172.72 53.34 0)
 			(hide yes)
@@
 			)
 		)
-		(property "LCSC Part #" "C427233"
+		(property "LCSC Part #" "C5736551"
 			(at 332.74 53.34 0)
 			(hide yes)
@@
 			)
 		)
-		(property "LCSC Part #" "C427231"
+		(property "LCSC Part #" "C313374"
 			(at 30.48 53.34 0)
 			(hide yes)
@@
 			)
 		)
-		(property "LCSC Part #" "C427233"
+		(property "LCSC Part #" "C5736551"
 			(at 190.5 53.34 0)
 			(hide yes)
@@
 			)
 		)
-		(property "LCSC Part #" "C427231"
+		(property "LCSC Part #" "C313374"
 			(at 101.6 53.34 0)
 			(hide yes)
@@
 			)
 		)
-		(property "LCSC Part #" "C427233"
+		(property "LCSC Part #" "C5736551"
 			(at 48.26 53.34 0)
 			(hide yes)
@@
 			)
 		)
-		(property "LCSC Part #" "C427231"
+		(property "LCSC Part #" "C313374"
 			(at 243.84 53.34 0)
 			(hide yes)
@@
 			)
 		)
-		(property "LCSC Part #" "C427231"
+		(property "LCSC Part #" "C313374"
 			(at 297.18 53.34 0)
 			(hide yes)
@@
 			)
 		)
-		(property "LCSC Part #" "C427231"
+		(property "LCSC Part #" "C313374"
 			(at 314.96 53.34 0)
 			(hide yes)
@@
 			)
 		)
-		(property "LCSC Part #" "C427233"
+		(property "LCSC Part #" "C5736551"
 			(at 137.16 53.34 0)
 			(hide yes)

Commit message: v0.4r2: conservative column resistors 47 Ω red / 100 Ω IR (~0.7 A per panel)
Red banks R_T0/R_T3: ROHM ESR01MZPF47R0 (C5736551); IR banks R_T1/R_T2:
Panasonic ERJ-PA2F1000X (C427235); both 0.2 W 0402. Model: red ≈52 mA
(57 % of rating, x2 vs v0.4r1), IR ≈33 mA (50 %, unchanged); all-on row
0.80 A, panel average ≈0.72 A, rail droop ≈0.40 V (stays above the
UCC27517 4.5 V minimum). Replaces the 22/47 Ω variant, which drew ≈1.2 A
per panel. Silkscreen legend "R: 47|100Ω"; production BOM, gerbers and
DRC report regenerated (schematic parity 0).

Co-Authored-By: Claude Fable 5.1 <noreply@anthropic.com>
Parts:
- R10, R11, R14, R15, R18, R19, R22, R23, R26, R27: LCSC Part # C5736551 -> C427235
- R12, R13, R16, R17, R20, R21, R24, R25, R28, R9: LCSC Part # C313374 -> C5736551
Changed lines of the file:
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@@
 			)
 		)
-		(property "LCSC Part #" "C313374"
+		(property "LCSC Part #" "C5736551"
 			(at 83.82 53.34 0)
 			(hide yes)
@@
 			)
 		)
-		(property "LCSC Part #" "C5736551"
+		(property "LCSC Part #" "C427235"
 			(at 66.04 53.34 0)
 			(hide yes)
@@
 			)
 		)
-		(property "LCSC Part #" "C313374"
+		(property "LCSC Part #" "C5736551"
 			(at 154.94 53.34 0)
 			(hide yes)
@@
 			)
 		)
-		(property "LCSC Part #" "C313374"
+		(property "LCSC Part #" "C5736551"
 			(at 369.57 53.34 0)
 			(hide yes)
@@
 			)
 		)
-		(property "LCSC Part #" "C5736551"
+		(property "LCSC Part #" "C427235"
 			(at 279.4 53.34 0)
 			(hide yes)
@@
 			)
 		)
-		(property "LCSC Part #" "C5736551"
+		(property "LCSC Part #" "C427235"
 			(at 261.62 53.34 0)
 			(hide yes)
@@
 			)
 		)
-		(property "LCSC Part #" "C5736551"
+		(property "LCSC Part #" "C427235"
 			(at 208.28 53.34 0)
 			(hide yes)
@@
 			)
 		)
-		(property "LCSC Part #" "C313374"
+		(property "LCSC Part #" "C5736551"
 			(at 226.06 53.34 0)
 			(hide yes)
@@
 			)
 		)
-		(property "LCSC Part #" "C5736551"
+		(property "LCSC Part #" "C427235"
 			(at 119.38 53.34 0)
 			(hide yes)
@@
 			)
 		)
-		(property "LCSC Part #" "C5736551"
+		(property "LCSC Part #" "C427235"
 			(at 351.79 53.34 0)
 			(hide yes)
@@
 			)
 		)
-		(property "LCSC Part #" "C313374"
+		(property "LCSC Part #" "C5736551"
 			(at 172.72 53.34 0)
 			(hide yes)
@@
 			)
 		)
-		(property "LCSC Part #" "C5736551"
+		(property "LCSC Part #" "C427235"
 			(at 332.74 53.34 0)
 			(hide yes)
@@
 			)
 		)
-		(property "LCSC Part #" "C313374"
+		(property "LCSC Part #" "C5736551"
 			(at 30.48 53.34 0)
 			(hide yes)
@@
 			)
 		)
-		(property "LCSC Part #" "C5736551"
+		(property "LCSC Part #" "C427235"
 			(at 190.5 53.34 0)
 			(hide yes)
@@
 			)
 		)
-		(property "LCSC Part #" "C313374"
+		(property "LCSC Part #" "C5736551"
 			(at 101.6 53.34 0)
 			(hide yes)
@@
 			)
 		)
-		(property "LCSC Part #" "C5736551"
+		(property "LCSC Part #" "C427235"
 			(at 48.26 53.34 0)
 			(hide yes)
@@
 			)
 		)
-		(property "LCSC Part #" "C313374"
+		(property "LCSC Part #" "C5736551"
 			(at 243.84 53.34 0)
 			(hide yes)
@@
 			)
 		)
-		(property "LCSC Part #" "C313374"
+		(property "LCSC Part #" "C5736551"
 			(at 297.18 53.34 0)
 			(hide yes)
@@
 			)
 		)
-		(property "LCSC Part #" "C313374"
+		(property "LCSC Part #" "C5736551"
 			(at 314.96 53.34 0)
 			(hide yes)
@@
 			)
 		)
-		(property "LCSC Part #" "C5736551"
+		(property "LCSC Part #" "C427235"
 			(at 137.16 53.34 0)
 			(hide yes)
