File: panel_rp2354_20x20_ir-red_v0p4/panel_rp2354_20x20.kicad_pcb (KiCad board)
At the start: 6 copper layers, 45 x 45 mm, 557 parts, among them J1 Conn_01x04, J2 Conn_01x05, J3 Conn_01x05, J4 Conn_01x05, J5 Conn_01x05, SW1 SW_Push, SW2 SW_Push, U1 APS6404L-3SQR, U10 UCC27517, U11 UCC27517, U12 UCC27517, U13 UCC27517, U14 UCC27517, U15 UCC27517, U16 UCC27517, U17 UCC27517, U18 UCC27517, U19 UCC27517, U2 RP2354B_80QFN, U20 UCC27517, U21 UCC27517, U22 UCC27517, U23 UCC27517, U24 UCC27517, U25 UCC27517, U26 UCC27517, U27 UCC27517, U28 UCC27517, U29 UCC27517, U3 UCC27517, U30 UCC27517, U31 UCC27517, U32 UCC27517, U33 UCC27517, U34 UCC27517, U35 UCC27517, U36 UCC27517, U37 UCC27517, U38 UCC27517, U39 UCC27517, U4 UCC27517, U40 UCC27517, U41 UCC27517, U42 UCC27517, U43 AP2112K-3.3, U5 UCC27517, U6 UCC27517, U7 UCC27517, U8 UCC27517, U9 UCC27517, Y1 ABM8-272-T3

Commit message: v0.4r2: fix all-on operating point, update silkscreen legend
- Operating point for the chosen 22/47 Ω pair recomputed together (was
  taken from 22/56 and 33/47 columns): all-on red 79 mA / IR 57 mA, row
  1.36 A, 5 V average 1.22 A (1.29 A RMS), droop 0.68 V -> ~4.3 V at the
  drivers vs UCC27517 4.5 V min VDD. Notes updated.
- B.SilkS legend: "R: 22|47Ω", "0|3: APHHS1005SURCK", "1|2: IN-S42CTQIR"
  (was 100Ω / 0|2 / 1|3). Gerbers and DRC report regenerated;
  schematic parity 0 issues.

Both found by the Codex cross-review.

Co-Authored-By: Claude Fable 5.1 <noreply@anthropic.com>
Other:
- board text added: "0|3: APHHS1005SURCK"
- board text added: "1|2: IN-S42CTQIR"
- board text added: "R: 22|47Ω"
- board text removed: "0|2: APHHS1005SURCK"
- board text removed: "1|3: IN-S42CTQIR"
- board text removed: "R: 100Ω ±1%"
Changed lines of the file:
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@@
 		(layer "Edge.Cuts")
 	)
-	(gr_text "R: 100Ω ±1%"
+	(gr_text "R: 22|47Ω"
 		(at 72.2 83.8 0)
 		(layer "B.SilkS")
@@
 		)
 	)
-	(gr_text "0|2: APHHS1005SURCK"
+	(gr_text "0|3: APHHS1005SURCK"
 		(at 78.4 67.2 0)
 		(layer "B.SilkS")
@@
 		)
 	)
-	(gr_text "1|3: IN-S42CTQIR"
+	(gr_text "1|2: IN-S42CTQIR"
 		(at 78.4 70.6 0)
 		(layer "B.SilkS")

Commit message: v0.4r2: conservative column resistors 47 Ω red / 100 Ω IR (~0.7 A per panel)
Red banks R_T0/R_T3: ROHM ESR01MZPF47R0 (C5736551); IR banks R_T1/R_T2:
Panasonic ERJ-PA2F1000X (C427235); both 0.2 W 0402. Model: red ≈52 mA
(57 % of rating, x2 vs v0.4r1), IR ≈33 mA (50 %, unchanged); all-on row
0.80 A, panel average ≈0.72 A, rail droop ≈0.40 V (stays above the
UCC27517 4.5 V minimum). Replaces the 22/47 Ω variant, which drew ≈1.2 A
per panel. Silkscreen legend "R: 47|100Ω"; production BOM, gerbers and
DRC report regenerated (schematic parity 0).

Co-Authored-By: Claude Fable 5.1 <noreply@anthropic.com>
Other:
- board text added: "R: 47|100Ω"
- board text removed: "R: 22|47Ω"
Changed lines of the file:
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@@
 			)
 		)
-		(property "LCSC Part #" "C5736551"
+		(property "LCSC Part #" "C427235"
 			(at 0 0 90)
 			(unlocked yes)
@@
 			)
 		)
-		(property "LCSC Part #" "C313374"
+		(property "LCSC Part #" "C5736551"
 			(at 0 0 90)
 			(unlocked yes)
@@
 			)
 		)
-		(property "LCSC Part #" "C313374"
+		(property "LCSC Part #" "C5736551"
 			(at 0 0 -90)
 			(unlocked yes)
@@
 			)
 		)
-		(property "LCSC Part #" "C313374"
+		(property "LCSC Part #" "C5736551"
 			(at 0 0 90)
 			(unlocked yes)
@@
 			)
 		)
-		(property "LCSC Part #" "C313374"
+		(property "LCSC Part #" "C5736551"
 			(at 0 0 90)
 			(unlocked yes)
@@
 			)
 		)
-		(property "LCSC Part #" "C313374"
+		(property "LCSC Part #" "C5736551"
 			(at 0 0 -90)
 			(unlocked yes)
@@
 			)
 		)
-		(property "LCSC Part #" "C5736551"
+		(property "LCSC Part #" "C427235"
 			(at 0 0 90)
 			(unlocked yes)
@@
 			)
 		)
-		(property "LCSC Part #" "C5736551"
+		(property "LCSC Part #" "C427235"
 			(at 0 0 -90)
 			(unlocked yes)
@@
 			)
 		)
-		(property "LCSC Part #" "C5736551"
+		(property "LCSC Part #" "C427235"
 			(at 0 0 90)
 			(unlocked yes)
@@
 			)
 		)
-		(property "LCSC Part #" "C313374"
+		(property "LCSC Part #" "C5736551"
 			(at 0 0 90)
 			(unlocked yes)
@@
 			)
 		)
-		(property "LCSC Part #" "C5736551"
+		(property "LCSC Part #" "C427235"
 			(at 0 0 90)
 			(unlocked yes)
@@
 			)
 		)
-		(property "LCSC Part #" "C313374"
+		(property "LCSC Part #" "C5736551"
 			(at 0 0 90)
 			(unlocked yes)
@@
 			)
 		)
-		(property "LCSC Part #" "C5736551"
+		(property "LCSC Part #" "C427235"
 			(at 0 0 90)
 			(unlocked yes)
@@
 			)
 		)
-		(property "LCSC Part #" "C313374"
+		(property "LCSC Part #" "C5736551"
 			(at 0 0 90)
 			(unlocked yes)
@@
 			)
 		)
-		(property "LCSC Part #" "C313374"
+		(property "LCSC Part #" "C5736551"
 			(at 0 0 90)
 			(unlocked yes)
@@
 			)
 		)
-		(property "LCSC Part #" "C5736551"
+		(property "LCSC Part #" "C427235"
 			(at 0 0 90)
 			(unlocked yes)
@@
 			)
 		)
-		(property "LCSC Part #" "C5736551"
+		(property "LCSC Part #" "C427235"
 			(at 0 0 90)
 			(unlocked yes)
@@
 			)
 		)
-		(property "LCSC Part #" "C313374"
+		(property "LCSC Part #" "C5736551"
 			(at 0 0 90)
 			(unlocked yes)
@@
 			)
 		)
-		(property "LCSC Part #" "C5736551"
+		(property "LCSC Part #" "C427235"
 			(at 0 0 90)
 			(unlocked yes)
@@
 			)
 		)
-		(property "LCSC Part #" "C5736551"
+		(property "LCSC Part #" "C427235"
 			(at 0 0 -90)
 			(unlocked yes)
@@
 		(layer "Edge.Cuts")
 	)
-	(gr_text "R: 22|47Ω"
+	(gr_text "R: 47|100Ω"
 		(at 72.2 83.8 0)
 		(layer "B.SilkS")
