File: panel_rp2354_20x20_four-color_v0p5/panel_rp2354_20x20.kicad_pcb (KiCad board)
At the start: 6 copper layers, 45 x 45 mm, 557 parts, among them J1 Conn_01x04, J2 Conn_01x05, J3 Conn_01x05, J4 Conn_01x05, J5 Conn_01x05, SW1 SW_Push, SW2 SW_Push, U1 APS6404L-3SQR, U10 UCC27517, U11 UCC27517, U12 UCC27517, U13 UCC27517, U14 UCC27517, U15 UCC27517, U16 UCC27517, U17 UCC27517, U18 UCC27517, U19 UCC27517, U2 RP2354B_80QFN, U20 UCC27517, U21 UCC27517, U22 UCC27517, U23 UCC27517, U24 UCC27517, U25 UCC27517, U26 UCC27517, U27 UCC27517, U28 UCC27517, U29 UCC27517, U3 UCC27517, U30 UCC27517, U31 UCC27517, U32 UCC27517, U33 UCC27517, U34 UCC27517, U35 UCC27517, U36 UCC27517, U37 UCC27517, U38 UCC27517, U39 UCC27517, U4 UCC27517, U40 UCC27517, U41 UCC27517, U42 UCC27517, U43 AP2112K-3.3, U5 UCC27517, U6 UCC27517, U7 UCC27517, U8 UCC27517, U9 UCC27517, Y1 ABM8-272-T3

Commit message: manual cleanup
Parts:
- moved C32 0.53 mm to (50.6, 63.8)
- moved R15 0.33 mm to (50.7, 78.8), turned to -90 degrees
- moved R21 0.29 mm to (50.6, 71.0)
- moved U21 0.15 mm to (67.4, 52.3)
- moved U17 0.10 mm to (67.3, 56.7)
- moved R10 0.09 mm to (55.0, 87.5)
- turned R22 to -90 degrees
- turned R14 to -90 degrees
Routing:
- net GND: track 260.3 -> 273.0 mm
- net Net-(D100-A): track 115.5 -> 123.4 mm
- net +5V: track 100.4 -> 106.6 mm, vias 57 -> 56
- net Net-(D101-A): track 125.8 -> 131.1 mm
- net /drivers/ROW_06: track 92.2 -> 97.0 mm
- net Net-(D181-A): track 142.5 -> 146.9 mm
- net Net-(D1-A): track 110.9 -> 114.5 mm, vias 17 -> 16
- net Net-(D141-A): track 125.9 -> 129.4 mm
- net Net-(D221-A): track 130.2 -> 133.4 mm
- net Net-(D261-A): track 144.7 -> 141.6 mm
- net Net-(D161-A): track 113.9 -> 117.0 mm
- net Net-(D41-A): track 114.5 -> 117.1 mm
- net Net-(D201-A): track 125.1 -> 127.7 mm
- net Net-(D241-A): track 140.0 -> 142.3 mm
- net +1V1: track 37.9 -> 40.1 mm
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
Commit message: DRC passes
Parts:
- moved R29 0.22 mm to (80.1, 73.4)
- moved C31 0.16 mm to (50.5, 68.6)
- moved R25 0.12 mm to (59.5, 66.4)
- moved U43 0.07 mm to (65.5, 92.5)
- moved R16 0.07 mm to (59.5, 75.0)
- moved R19 0.06 mm to (59.5, 70.7)
- moved R26 0.06 mm to (55.1, 66.4)
- moved R9 0.06 mm to (59.5, 87.5), turned to -90 degrees
Routing:
- net Net-(D61-A): track 104.8 -> 118.7 mm, vias 13 -> 14
- net +5V: track 106.6 -> 94.7 mm, vias 56 -> 53
- net GND: track 273.0 -> 266.6 mm, vias 72 -> 68
- net Net-(D101-A): track 131.1 -> 126.5 mm
- net Net-(D341-A): track 143.6 -> 147.7 mm
- net Net-(D321-A): track 153.2 -> 149.1 mm
- net Net-(D361-A): track 152.0 -> 156.0 mm
- net Net-(D281-A): track 122.4 -> 126.1 mm
- net Net-(D141-A): track 129.4 -> 132.9 mm
- net Net-(D381-A): track 121.1 -> 124.4 mm
- net Net-(D201-A): track 127.7 -> 130.8 mm
- net /drivers/ROW_MCU_04: track 22.7 -> 25.4 mm
- net Net-(D121-A): track 110.2 -> 112.7 mm
- net /drivers/ROW_MCU_12: track 22.5 -> 24.7 mm
- net Net-(D301-A): track 128.8 -> 130.8 mm
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