File: panel_rp2354_20x20_four-color_v0p5/panel_mcu.kicad_sch (KiCad schematic)
At the start: 33 parts, among them SW1 SW_Push, SW2 SW_Push, U1 APS6404L-3SQR, U2 RP2354B_80QFN, Y1 ABM8-272-T3

Commit message: add DBG connector
Parts:
- added J6: Conn_01x03, Connector_JST:JST_SH_BM03B-SRSS-TB_1x03-1MP_P1.00mm_Vertical, symbol Connector_Generic:Conn_01x03
Connections:
- net GND: now also J6.2 (Pin_2)
- net at U2.33 (SWCLK): now also J6.1 (Pin_1)
- net at U2.34 (SWD): now also J6.3 (Pin_3)
- no-connect marks 4 -> 2
